Commit message: feat(camera): topic-controllable movable 4K camera + calibration tooling
- teleop: move camera over /gazebo/set_model_state topic (drop service);
  fix dropped keypresses with stdbuf; drone Mode-2 key mapping
- urdf: parameterize <static>; movable (gravity-off) mode so set_model_state
  can relocate the camera; default resolution bumped to 4K (3840x2160 @ 15fps)
- models/usb_cam: reusable non-static SDF camera model (sensor +
  libgazebo_ros_camera) for model:// spawning and GAZEBO_MODEL_PATH
- web_calibration: browser intrinsic calibrator reusing camera_calibration
  MonoCalibrator (MJPEG stream, 3D sample guide, reference snapshots,
  auto-run) -- to be relocated to the perception layer in a later step
- update launches, tests, README, CMakeLists, compliance accordingly

Co-Authored-By: Claude Opus 4.8 (1M context) <noreply@anthropic.com>
Claude-Session: https://claude.ai/code/session_018bY65i7hdP86C2u3jgDuqZ

File: urdf/checkerboard_8x6.urdf.xacro (robot description, xacro)
@@ -5,9 +5,26 @@
   <xacro:property name="s" value="0.20"/>
   <xacro:macro name="black_square" params="column row">
-    <visual>
+    <link name="checker_black_${column}_${row}">
+      <inertial>
+        <mass value="0.001"/>
+        <inertia ixx="0.00000667" ixy="0" ixz="0"
+                 iyy="0.00000334" iyz="0" izz="0.00000334"/>
+      </inertial>
+      <visual>
+        <geometry><box size="0.004 ${s} ${s}"/></geometry>
+        <material name="black"><color rgba="0.01 0.01 0.01 1"/></material>
+      </visual>
+    </link>
+    <joint name="checker_black_${column}_${row}_joint" type="fixed">
+      <parent link="board"/>
+      <child link="checker_black_${column}_${row}"/>
       <origin xyz="-0.011 ${(-0.7 + 0.2*column)} ${(-0.5 + 0.2*row)}"/>
-      <geometry><box size="0.004 ${s} ${s}"/></geometry>
-      <material name="black"><color rgba="0.01 0.01 0.01 1"/></material>
-    </visual>
+    </joint>
+    <gazebo reference="checker_black_${column}_${row}">
+      <material>Gazebo/Black</material>
+    </gazebo>
+    <gazebo reference="checker_black_${column}_${row}_joint">
+      <preserveFixedJoint>true</preserveFixedJoint>
+    </gazebo>
   </xacro:macro>
   <!-- Eight by six squares, i.e. seven by five internal calibration corners. -->
@@ -19,11 +36,12 @@
     </visual>
     <collision><geometry><box size="0.02 1.60 1.20"/></geometry></collision>
-    <xacro:black_square column="0" row="0"/><xacro:black_square column="2" row="0"/><xacro:black_square column="4" row="0"/><xacro:black_square column="6" row="0"/>
-    <xacro:black_square column="1" row="1"/><xacro:black_square column="3" row="1"/><xacro:black_square column="5" row="1"/><xacro:black_square column="7" row="1"/>
-    <xacro:black_square column="0" row="2"/><xacro:black_square column="2" row="2"/><xacro:black_square column="4" row="2"/><xacro:black_square column="6" row="2"/>
-    <xacro:black_square column="1" row="3"/><xacro:black_square column="3" row="3"/><xacro:black_square column="5" row="3"/><xacro:black_square column="7" row="3"/>
-    <xacro:black_square column="0" row="4"/><xacro:black_square column="2" row="4"/><xacro:black_square column="4" row="4"/><xacro:black_square column="6" row="4"/>
-    <xacro:black_square column="1" row="5"/><xacro:black_square column="3" row="5"/><xacro:black_square column="5" row="5"/><xacro:black_square column="7" row="5"/>
   </link>
+  <gazebo reference="board"><material>Gazebo/White</material></gazebo>
+  <xacro:black_square column="0" row="0"/><xacro:black_square column="2" row="0"/><xacro:black_square column="4" row="0"/><xacro:black_square column="6" row="0"/>
+  <xacro:black_square column="1" row="1"/><xacro:black_square column="3" row="1"/><xacro:black_square column="5" row="1"/><xacro:black_square column="7" row="1"/>
+  <xacro:black_square column="0" row="2"/><xacro:black_square column="2" row="2"/><xacro:black_square column="4" row="2"/><xacro:black_square column="6" row="2"/>
+  <xacro:black_square column="1" row="3"/><xacro:black_square column="3" row="3"/><xacro:black_square column="5" row="3"/><xacro:black_square column="7" row="3"/>
+  <xacro:black_square column="0" row="4"/><xacro:black_square column="2" row="4"/><xacro:black_square column="4" row="4"/><xacro:black_square column="6" row="4"/>
+  <xacro:black_square column="1" row="5"/><xacro:black_square column="3" row="5"/><xacro:black_square column="5" row="5"/><xacro:black_square column="7" row="5"/>
   <gazebo><static>true</static></gazebo>
 </robot>

File: urdf/fixed_rgb_camera.urdf.xacro (robot description, xacro)
@@ -12,11 +12,18 @@
   <xacro:arg name="camera_link_frame" default="usb_cam_link"/>
   <xacro:arg name="optical_frame" default="usb_cam_optical_frame"/>
-  <xacro:arg name="width" default="1920"/>
-  <xacro:arg name="height" default="1080"/>
-  <xacro:arg name="fps" default="30.0"/>
+  <xacro:arg name="width" default="3840"/>
+  <xacro:arg name="height" default="2160"/>
+  <xacro:arg name="fps" default="15.0"/>
   <xacro:arg name="hfov" default="1.3962634"/>
   <xacro:arg name="near_clip" default="0.05"/>
   <xacro:arg name="far_clip" default="100.0"/>
   <xacro:arg name="noise_stddev" default="0.0"/>
+  <xacro:arg name="static" default="true"/>
+  <!-- Compact black camera body: x is the optical/forward axis. -->
+  <xacro:property name="body_depth" value="0.06"/>
+  <xacro:property name="body_side" value="0.14"/>
+  <xacro:property name="lens_length" value="0.035"/>
+  <xacro:property name="lens_radius" value="0.04"/>
+  <xacro:property name="lens_center_x" value="${(body_depth + lens_length) / 2.0}"/>
   <link name="$(arg camera_link_frame)">
     <inertial>
@@ -26,8 +33,19 @@
     </inertial>
     <visual>
-      <geometry><box size="0.12 0.18 0.10"/></geometry>
-      <material name="camera_dark"><color rgba="0.08 0.08 0.08 1"/></material>
+      <geometry><box size="${body_depth} ${body_side} ${body_side}"/></geometry>
+      <material name="camera_black"><color rgba="0.02 0.02 0.02 1"/></material>
     </visual>
-    <collision><geometry><box size="0.12 0.18 0.10"/></geometry></collision>
+    <visual>
+      <origin xyz="${lens_center_x} 0 0" rpy="0 ${pi/2} 0"/>
+      <geometry><cylinder radius="${lens_radius}" length="${lens_length}"/></geometry>
+      <material name="camera_black"/>
+    </visual>
+    <collision>
+      <geometry><box size="${body_depth} ${body_side} ${body_side}"/></geometry>
+    </collision>
+    <collision>
+      <origin xyz="${lens_center_x} 0 0" rpy="0 ${pi/2} 0"/>
+      <geometry><cylinder radius="${lens_radius}" length="${lens_length}"/></geometry>
+    </collision>
   </link>
   <link name="$(arg optical_frame)"/>
@@ -38,7 +56,21 @@
     <origin xyz="0 0 0" rpy="${-pi/2} 0 ${-pi/2}"/>
   </joint>
-  <!-- Model-level static flag: the fixed-site camera must never fall. -->
-  <gazebo><static>true</static></gazebo>
+  <!--
+    Fixed-site default (static:=true): the camera is pinned so it never falls.
+    Movable mode (static:=false, used by the calibration/teleop world): the
+    model stays in the physics engine so /gazebo/set_model_state can reposition
+    it, while per-link gravity is disabled so it floats in place instead of
+    falling.  A <static>true</static> model is excluded from physics entirely,
+    so set_model_state silently fails to move it (and the render never changes).
+  -->
+  <xacro:if value="$(arg static)">
+    <gazebo><static>true</static></gazebo>
+  </xacro:if>
+  <xacro:unless value="$(arg static)">
+    <gazebo reference="$(arg camera_link_frame)"><gravity>false</gravity></gazebo>
+  </xacro:unless>
   <gazebo reference="$(arg camera_link_frame)">
+    <!-- Gazebo Classic does not reliably preserve URDF RGBA colors. -->
+    <material>Gazebo/Black</material>
     <sensor name="rgb_camera" type="camera">
       <always_on>true</always_on>
